File: kicad/Z80_CPU.kicad_sch (KiCad schematic)
At the start: 106 parts, among them J101 Conn_01x10, J106 Conn_01x10, J2 C96ABC, J3 DIN-5, J39 Conn_01x04, U71 CDB407, U72 CDB407, U73 CDB407, U74 CDB407, U90 Z80CPU

Commit message: add doc folder, ro and en readme
Parts:
- JP3: value bA14 -> bA15
- JP3: value bA14 -> nRST
Changed lines of the file:
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@@
       (effects (font (size 1.27 1.27)))
     )
-    (property "Value" "bA14" (at 110.49 143.51 0)
+    (property "Value" "bA15" (at 110.49 143.51 0)
       (effects (font (size 1.27 1.27)))
     )
@@
       (effects (font (size 1.27 1.27)))
     )
-    (property "Value" "bA14" (at 110.49 147.955 0)
-      (effects (font (size 1.27 1.27)))
-    )
+    (property "Value" "nRST" (at 110.49 147.955 0)
+      (effects (font (size 1.27 1.27)))
+    )
